File: kicad/usb_c_traffic_light_board.kicad_sch (KiCad schematic)
At the start: 0 parts

Commit message: 提交红绿灯控制板阶段性设计
Other:
- note added: "12 P3.6/UDP <- USB D+"
- note added: "13 P3.7/UDM <- USB D-"
- note added: "14 GND"
- note added: "15 VCC -> 5V"
- note added: "16 V33 -> C3 100nF 到地"
- note added: "2 P1.4 -> 红灯"
- note added: "3 P1.5 -> 黄灯"
- note added: "4 P1.6 -> 绿灯"
- note added: "5V"
- note added: "6 RST -> 测试焊盘"
- note added: "C1 10uF"
- note added: "C2 100nF"
- note added: "C3 100nF"
- note added: "CC1: A5"
- note added: "CC2: B5"
- note added: "D+: A6/B6"
- note added: "D-: A7/B7"
- note added: "D1 绿灯"
- note added: "D2 黄灯"
- note added: "D3 红灯"
- note added: "GND"
- note added: "GND: A1/B1/A12/B12"
- note added: "J1 USB-C 母座"
- note added: "R1 1k"
- note added: "R2 1k"
- note added: "R3 1k"
- note added: "R4 22Ω"
- note added: "R5 22Ω"
- note added: "R6 5.1k"
- note added: "R7 5.1k"
- note added: "TP：5V / GND / D+ / D- / RST / 红灯 / 黄灯 / 绿灯"
- note added: "U1 CH552G SOP-16"
- note added: "USB-C 红绿灯控制板完整原理图（第一版）"
- note added: "VBUS: A4/B4/A9/B9"
- note added: "三路 LED 阴极接地；GPIO 高电平点亮"
- note added: "说明：这是可在 KiCad 原理图编辑器中直接看到的连接图；下一版再替换为正式符号库器件。"
- note removed: "原理图草案。选定 USB-C 母座和 CH552G KiCad 符号后补全器件。"
Changed lines of the file:
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@@
 (kicad_sch
-  (version 20231120)
-  (generator "codex")
-  (generator_version "1")
+  (version 20250610)
+  (generator "eeschema")
+  (generator_version "10.0")
   (paper "A4")
   (title_block
     (title "USB-C 红绿灯控制板")
     (date "2026-05-25")
-    (rev "A-draft")
+    (rev "A1")
     (company "lemonhall")
-    (comment 1 "CH552G USB 串口控制红黄绿三颗灯")
+    (comment 1 "CH552G 通过 USB 串口控制红黄绿三颗灯")
   )
-  (text "原理图草案。选定 USB-C 母座和 CH552G KiCad 符号后补全器件。"
-    (exclude_from_sim no)
-    (at 40 40 0)
-    (effects (font (size 1.27 1.27)) (justify left bottom))
+  (text "USB-C 红绿灯控制板完整原理图（第一版）" (at 18 18 0)
+    (effects (font (size 3.0 3.0) (bold yes)) (justify left bottom))
+)
+  (text "说明：这是可在 KiCad 原理图编辑器中直接看到的连接图；下一版再替换为正式符号库器件。" (at 18 25 0)
+    (effects (font (size 1.6 1.6)) (justify left bottom))
+)
+  (polyline (pts (xy 18 42) (xy 64 42) (xy 64 112) (xy 18 112) (xy 18 42))
+    (stroke (width 0.25) (type solid))
+    (fill (type none))
+)
+  (text "J1 USB-C 母座" (at 24 49 0)
+    (effects (font (size 1.8 1.8) (bold yes)) (justify left bottom))
+)
+  (text "VBUS: A4/B4/A9/B9" (at 24 58 0) (effects (font (size 1.35 1.35)) (justify left bottom)))
+  (text "GND: A1/B1/A12/B12" (at 24 65 0) (effects (font (size 1.35 1.35)) (justify left bottom)))
+  (text "D+: A6/B6" (at 24 72 0) (effects (font (size 1.35 1.35)) (justify left bottom)))
+  (text "D-: A7/B7" (at 24 79 0) (effects (font (size 1.35 1.35)) (justify left bottom)))
+  (text "CC1: A5" (at 24 86 0) (effects (font (size 1.35 1.35)) (justify left bottom)))
+  (text "CC2: B5" (at 24 93 0) (effects (font (size 1.35 1.35)) (justify left bottom)))
+  (polyline (pts (xy 93 36) (xy 150 36) (xy 150 126) (xy 93 126) (xy 93 36))
+    (stroke (width 0.25) (type solid))
+    (fill (type none))
+)
+  (text "U1 CH552G SOP-16" (at 104 44 0)
+    (effects (font (size 1.8 1.8) (bold yes)) (justify left bottom))
+)
+  (text "15 VCC -> 5V" (at 100 55 0) (effects (font (size 1.35 1.35)) (justify left bottom)))
+  (text "16 V33 -> C3 100nF 到地" (at 100 62 0) (effects (font (size 1.35 1.35)) (justify left bottom)))
+  (text "14 GND" (at 100 69 0) (effects (font (size 1.35 1.35)) (justify left bottom)))
+  (text "12 P3.6/UDP <- USB D+" (at 100 80 0) (effects (font (size 1.35 1.35)) (justify left bottom)))
+  (text "13 P3.7/UDM <- USB D-" (at 100 87 0) (effects (font (size 1.35 1.35)) (justify left bottom)))
+  (text "2 P1.4 -> 红灯" (at 100 99 0) (effects (font (size 1.35 1.35)) (justify left bottom)))
+  (text "3 P1.5 -> 黄灯" (at 100 106 0) (effects (font (size 1.35 1.35)) (justify left bottom)))
+  (text "4 P1.6 -> 绿灯" (at 100 113 0) (effects (font (size 1.35 1.35)) (justify left bottom)))
+  (text "6 RST -> 测试焊盘" (at 100 120 0) (effects (font (size 1.35 1.35)) (justify left bottom)))
+  (polyline (pts (xy 74 78) (xy 88 78) (xy 88 85) (xy 74 85) (xy 74 78))
+    (stroke (width 0.2) (type solid))
+    (fill (type none))
+)
+  (text "R4 22Ω" (at 75 83 0) (effects (font (size 1.1 1.1)) (justify left bottom)))
+  (polyline (pts (xy 74 88) (xy 88 88) (xy 88 95) (xy 74 95) (xy 74 88))
+    (stroke (width 0.2) (type solid))
+    (fill (type none))
+)
+  (text "R5 22Ω" (at 75 93 0) (effects (font (size 1.1 1.1)) (justify left bottom)))
+  (polyline (pts (xy 74 101) (xy 90 101) (xy 90 108) (xy 74 108) (xy 74 101))
+    (stroke (width 0.2) (type solid))
+    (fill (type none))
+)
+  (text "R6 5.1k" (at 75 106 0) (effects (font (size 1.1 1.1)) (justify left bottom)))
+  (polyline (pts (xy 74 113) (xy 90 113) (xy 90 120) (xy 74 120) (xy 74 113))
+    (stroke (width 0.2) (type solid))
+    (fill (type none))
+)
+  (text "R7 5.1k" (at 75 118 0) (effects (font (size 1.1 1.1)) (justify left bottom)))
+  (polyline (pts (xy 174 50) (xy 202 50) (xy 202 62) (xy 174 62) (xy 174 50))
+    (stroke (width 0.2) (type solid))
+    (fill (type none))
+)
+  (text "R1 1k" (at 181 58 0) (effects (font (size 1.3 1.3)) (justify left bottom)))
+  (polyline (pts (xy 214 50) (xy 246 50) (xy 246 62) (xy 214 62) (xy 214 50))
+    (stroke (width 0.2) (type solid))
+    (fill (type none))
+)
+  (text "D3 红灯" (at 221 58 0) (effects (font (size 1.3 1.3) (bold yes)) (justify left bottom)))
+  (polyline (pts (xy 174 75) (xy 202 75) (xy 202 87) (xy 174 87) (xy 174 75))
+    (stroke (width 0.2) (type solid))
+    (fill (type none))
+)
+  (text "R2 1k" (at 181 83 0) (effects (font (size 1.3 1.3)) (justify left bottom)))
+  (polyline (pts (xy 214 75) (xy 246 75) (xy 246 87) (xy 214 87) (xy 214 75))
+    (stroke (width 0.2) (type solid))
+    (fill (type none))
+)
+  (text "D2 黄灯" (at 221 83 0) (effects (font (size 1.3 1.3) (bold yes)) (justify left bottom)))
+  (polyline (pts (xy 174 100) (xy 202 100) (xy 202 112) (xy 174 112) (xy 174 100))
+    (stroke (width 0.2) (type solid))
+    (fill (type none))
+)
+  (text "R3 1k" (at 181 108 0) (effects (font (size 1.3 1.3)) (justify left bottom)))
+  (polyline (pts (xy 214 100) (xy 246 100) (xy 246 112) (xy 214 112) (xy 214 100))
+    (stroke (width 0.2) (type solid))
+    (fill (type none))
+)
+  (text "D1 绿灯" (at 221 108 0) (effects (font (size 1.3 1.3) (bold yes)) (justify left bottom)))
+  (polyline (pts (xy 76 140) (xy 104 140) (xy 104 152) (xy 76 152) (xy 76 140))
+    (stroke (width 0.2) (type solid))
+    (fill (type none))
+)
+  (text "C1 10uF" (at 83 148 0) (effects (font (size 1.3 1.3)) (justify left bottom)))
+  (polyline (pts (xy 118 140) (xy 150 140) (xy 150 152) (xy 118 152) (xy 118 140))
+    (stroke (width 0.2) (type solid))
+    (fill (type none))
+)
+  (text "C2 100nF" (at 123 148 0) (effects (font (size 1.3 1.3)) (justify left bottom)))
+  (polyline (pts (xy 166 140) (xy 198 140) (xy 198 152) (xy 166 152) (xy 166 140))
+    (stroke (width 0.2) (type solid))
+    (fill (type none))
+)
+  (text "C3 100nF" (at 171 148 0) (effects (font (size 1.3 1.3)) (justify left bottom)))
+  (wire (pts (xy 64 58) (xy 93 58)) (stroke (width 0.25) (type solid)))
+  (text "5V" (at 69 56 0) (effects (font (size 1.2 1.2)) (justify left bottom)))
+  (wire (pts (xy 64 65) (xy 93 69)) (stroke (width 0.25) (type solid)))
+  (text "GND" (at 69 66 0) (effects (font (size 1.2 1.2)) (justify left bottom)))
+  (wire (pts (xy 64 72) (xy 74 81.5)) (stroke (width 0.25) (type solid)))
+  (wire (pts (xy 88 81.5) (xy 93 80)) (stroke (width 0.25) (type solid)))
+  (wire (pts (xy 64 79) (xy 74 91.5)) (stroke (width 0.25) (type solid)))
+  (wire (pts (xy 88 91.5) (xy 93 87)) (stroke (width 0.25) (type solid)))
+  (wire (pts (xy 64 86) (xy 74 104.5)) (stroke (width 0.25) (type solid)))
+  (wire (pts (xy 90 104.5) (xy 90 126)) (stroke (width 0.25) (type solid)))
+  (wire (pts (xy 64 93) (xy 74 116.5)) (stroke (width 0.25) (type solid)))
+  (wire (pts (xy 90 116.5) (xy 90 126)) (stroke (width 0.25) (type solid)))
+  (text "GND" (at 88 132 0) (effects (font (size 1.2 1.2)) (justify left bottom)))
+  (wire (pts (xy 150 99) (xy 174 56)) (stroke (width 0.25) (type solid)))
+  (wire (pts (xy 202 56) (xy 214 56)) (stroke (width 0.25) (type solid)))
+  (wire (pts (xy 246 56) (xy 258 56)) (stroke (width 0.25) (type solid)))
+  (wire (pts (xy 258 56) (xy 258 126)) (stroke (width 0.25) (type solid)))
+  (wire (pts (xy 150 106) (xy 174 81)) (stroke (width 0.25) (type solid)))
+  (wire (pts (xy 202 81) (xy 214 81)) (stroke (width 0.25) (type solid)))
+  (wire (pts (xy 246 81) (xy 258 81)) (stroke (width 0.25) (type solid)))
+  (wire (pts (xy 150 113) (xy 174 106)) (stroke (width 0.25) (type solid)))
+  (wire (pts (xy 202 106) (xy 214 106)) (stroke (width 0.25) (type solid)))
+  (wire (pts (xy 246 106) (xy 258 106)) (stroke (width 0.25) (type solid)))
+  (text "三路 LED 阴极接地；GPIO 高电平点亮" (at 172 126 0) (effects (font (size 1.25 1.25)) (justify left bottom)))
+  (text "TP：5V / GND / D+ / D- / RST / 红灯 / 黄灯 / 绿灯" (at 18 168 0)
+    (effects (font (size 1.5 1.5) (bold yes)) (justify left bottom))
+)
+  (sheet_instances
+    (path "/" (page "1"))
   )
 )
